File: MINI_STM.kicad_sch (KiCad schematic)
At the start: 33 parts, among them J1 Programming, SW1 SW_Push, U1 STM32G431KBTx, U2 TPS565208

Commit message: Added more connectors and a power test point.
Parts:
- removed JP1: OSC_IN JP, symbol Jumper:SolderJumper_2_Bridged
- removed JP2: OSC_OUT JP, symbol Jumper:SolderJumper_2_Bridged
- added J2: POWER INPUT, symbol Connector:Screw_Terminal_01x02
- added J3: GPIO Connector, symbol Connector:Conn_01x10_Pin
- added JP1: OSC_IN JP, symbol Jumper:Jumper_2_Open
- added JP2: OSC_OUT JP, symbol Jumper:Jumper_2_Open
- added TP1: +3V3 TP, symbol Connector:TestPoint
Connections:
- net +3V3: now also TP1.1
- net GND: now also J2.1 (Pin_1)
- net OSC_IN: now also JP1.1 (A)
- net OSC_OUT: now also JP2.1 (A)
- net VIN (+12V): now also J2.2 (Pin_2)
- net PA5_IO: now reaches U1.10 (PA5)
- net PA5_IO: now also J3.6 (Pin_6)
- net PA6_IO: now reaches U1.11 (PA6)
- net PA6_IO: now also J3.7 (Pin_7)
- net PA7_IO: now reaches U1.12 (PA7)
- net PA7_IO: now also J3.8 (Pin_8)
- net PA8_IO: now reaches U1.18 (PA8)
- net PA8_IO: now also J3.9 (Pin_9)
- net PA9_IO: now reaches U1.19 (PA9)
- net PA9_IO: now also J3.10 (Pin_10)
- net at U1.2 (PF0): now also JP1.2 (B)
- net at U1.3 (PF1): now also JP2.2 (B)
- net PA0_IO: now reaches U1.5 (PA0)
- net PA0_IO: now also J3.1 (Pin_1)
- net PA1_IO: now reaches U1.6 (PA1)
- net PA1_IO: now also J3.2 (Pin_2)
- net PA2_IO: now reaches U1.7 (PA2)
- net PA2_IO: now also J3.3 (Pin_3)
- net PA3_IO: now reaches U1.8 (PA3)
- net PA3_IO: now also J3.4 (Pin_4)
- net PA4_IO: now reaches U1.9 (PA4)
- net PA4_IO: now also J3.5 (Pin_5)
- no-connect marks 23 -> 13
Other:
- moved on the sheet: C10, C11, C12, C13, C14, C7, C8, C9, D1, D2, FB1, J1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

Commit message: Starting PCB layout.
Parts:
- C1, C2, C3, C4, C5, C6: footprint (none) -> Capacitor_SMD:C_0805_2012Metric_Pad1.18x1.45mm_HandSolder
- D2: footprint (none) -> LED_SMD:LED_0805_2012Metric_Pad1.15x1.40mm_HandSolder
- R1, R2, R3, R8: footprint (none) -> Resistor_SMD:R_0805_2012Metric_Pad1.20x1.40mm_HandSolder
- TP1: footprint (none) -> TestPoint:TestPoint_Pad_D4.0mm
Changed lines of the file:
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@@
 			)
 		)
-		(property "Footprint" ""
+		(property "Footprint" "Capacitor_SMD:C_0805_2012Metric_Pad1.18x1.45mm_HandSolder"
 			(at 37.7952 180.34 0)
 			(effects
@@
 			)
 		)
-		(property "Footprint" ""
+		(property "Footprint" "LED_SMD:LED_0805_2012Metric_Pad1.15x1.40mm_HandSolder"
 			(at 259.08 156.21 0)
 			(effects
@@
 			)
 		)
-		(property "Footprint" ""
+		(property "Footprint" "Resistor_SMD:R_0805_2012Metric_Pad1.20x1.40mm_HandSolder"
 			(at 64.77 175.768 90)
 			(effects
@@
 			)
 		)
-		(property "Footprint" ""
+		(property "Footprint" "Resistor_SMD:R_0805_2012Metric_Pad1.20x1.40mm_HandSolder"
 			(at 93.472 179.07 90)
 			(effects
@@
 			)
 		)
-		(property "Footprint" ""
+		(property "Footprint" "Capacitor_SMD:C_0805_2012Metric_Pad1.18x1.45mm_HandSolder"
 			(at 127.9652 163.83 0)
 			(effects
@@
 			)
 		)
-		(property "Footprint" ""
+		(property "Footprint" "Capacitor_SMD:C_0805_2012Metric_Pad1.18x1.45mm_HandSolder"
 			(at 96.8248 160.02 0)
 			(effects
@@
 			)
 		)
-		(property "Footprint" ""
+		(property "Footprint" "Resistor_SMD:R_0805_2012Metric_Pad1.20x1.40mm_HandSolder"
 			(at 109.22 175.768 90)
 			(effects
@@
 			)
 		)
-		(property "Footprint" ""
+		(property "Footprint" "Capacitor_SMD:C_0805_2012Metric_Pad1.18x1.45mm_HandSolder"
 			(at 49.2252 180.34 0)
 			(effects
@@
 			)
 		)
-		(property "Footprint" ""
+		(property "Footprint" "Resistor_SMD:R_0805_2012Metric_Pad1.20x1.40mm_HandSolder"
 			(at 246.38 157.988 90)
 			(effects
@@
 			)
 		)
-		(property "Footprint" ""
+		(property "Footprint" "TestPoint:TestPoint_Pad_D4.0mm"
 			(at 148.59 154.94 0)
 			(effects
@@
 			)
 		)
-		(property "Footprint" ""
+		(property "Footprint" "Capacitor_SMD:C_0805_2012Metric_Pad1.18x1.45mm_HandSolder"
 			(at 26.3652 180.34 0)
 			(effects
@@
 			)
 		)
-		(property "Footprint" ""
+		(property "Footprint" "Capacitor_SMD:C_0805_2012Metric_Pad1.18x1.45mm_HandSolder"
 			(at 116.5352 163.83 0)
 			(effects
